File: Hardware/WheelPod.sch (KiCad schematic (older format))
At the start: 0 parts

Commit message: Simple schematic/board for sizing purposes
Parts:
- added C1, C2: C, ~, symbol C
- added L1: L, ~, symbol L
- added U1: PIC32MX250F128D, ~, symbol PIC32MX250F128D
- added U2: LDC1000, ~, symbol LDC1000
Connections:
- new net: C1.2, L1.1, U2.10 (INB)
- new net: C2.2, U2.7 (CFB)
- new net: C2.1, U2.8 (CFA)
- new net: C1.1, L1.2, U2.9 (INA)
Changed lines of the file:
@@
 LIBS:power
 LIBS:Aerodyne_v2
+LIBS:WheelPod-cache
 EELAYER 27 0
 EELAYER END
@@
 Comment4 ""
 $EndDescr
+$Comp
+L PIC32MX250F128D U1
+U 1 1 5287E978
+P 1100 1000
+F 0 "U1" H 1050 1100 60  0000 C CNN
+F 1 "PIC32MX250F128D" V 850 500 60  0000 C CNN
+F 2 "~" H 1100 1000 60  0000 C CNN
+F 3 "~" H 1100 1000 60  0000 C CNN
+	1    1100 1000
+	1    0    0    -1
+$EndComp
+$Comp
+L PIC32MX250F128D U1
+U 2 1 5287E987
+P 1100 2400
+F 0 "U1" H 1050 2500 60  0000 C CNN
+F 1 "PIC32MX250F128D" V 850 1900 60  0000 C CNN
+F 2 "~" H 1100 2400 60  0000 C CNN
+F 3 "~" H 1100 2400 60  0000 C CNN
+	2    1100 2400
+	1    0    0    -1
+$EndComp
+$Comp
+L PIC32MX250F128D U1
+U 3 1 5287E996
+P 1100 3800
+F 0 "U1" H 1050 3900 60  0000 C CNN
+F 1 "PIC32MX250F128D" V 850 3300 60  0000 C CNN
+F 2 "~" H 1100 3800 60  0000 C CNN
+F 3 "~" H 1100 3800 60  0000 C CNN
+	3    1100 3800
+	1    0    0    -1
+$EndComp
+$Comp
+L PIC32MX250F128D U1
+U 4 1 5287E9A5
+P 1100 5200
+F 0 "U1" H 1050 5300 60  0000 C CNN
+F 1 "PIC32MX250F128D" V 850 4700 60  0000 C CNN
+F 2 "~" H 1100 5200 60  0000 C CNN
+F 3 "~" H 1100 5200 60  0000 C CNN
+	4    1100 5200
+	1    0    0    -1
+$EndComp
+$Comp
+L LDC1000 U2
+U 1 1 5287E9D6
+P 5100 2900
+F 0 "U2" H 5100 3400 60  0000 C CNN
+F 1 "LDC1000" V 5100 2900 60  0000 C CNN
+F 2 "~" H 5100 2900 60  0000 C CNN
+F 3 "~" H 5100 2900 60  0000 C CNN
+	1    5100 2900
+	1    0    0    -1
+$EndComp
+$Comp
+L L L1
+U 1 1 5287F733
+P 6500 2250
+F 0 "L1" H 6500 2150 60  0000 C CNN
+F 1 "L" H 6500 2300 60  0000 C CNN
+F 2 "~" H 6500 2250 60  0000 C CNN
+F 3 "~" H 6500 2250 60  0000 C CNN
+	1    6500 2250
+	0    -1   -1   0
+$EndComp
+$Comp
+L C C1
+U 1 1 5287F742
+P 6100 2250
+F 0 "C1" H 6150 2400 60  0000 L CNN
+F 1 "C" H 6150 2100 60  0000 L CNN
+F 2 "~" H 6100 2250 60  0000 C CNN
+F 3 "~" H 6100 2250 60  0000 C CNN
+F 4 "V" H 6050 2100 60  0001 R CNN "Voltage"
+F 5 "D" H 6050 2400 60  0001 R CNN "Dielectric"
+	1    6100 2250
+	-1   0    0    -1
+$EndComp
+Wire Wire Line
+	6100 2000 6100 1900
+Wire Wire Line
+	5700 1900 6500 1900
+Wire Wire Line
+	6500 1900 6500 2000
+Wire Wire Line
+	6500 2600 6500 2500
+Wire Wire Line
+	5600 2600 6500 2600
+Wire Wire Line
+	6100 2600 6100 2500
+$Comp
+L C C2
+U 1 1 5287F78E
+P 6500 3050
+F 0 "C2" H 6550 3200 60  0000 L CNN
+F 1 "C" H 6550 2900 60  0000 L CNN
+F 2 "~" H 6500 3050 60  0000 C CNN
+F 3 "~" H 6500 3050 60  0000 C CNN
+F 4 "V" H 6450 2900 60  0001 R CNN "Voltage"
+F 5 "D" H 6450 3200 60  0001 R CNN "Dielectric"
+	1    6500 3050
+	1    0    0    -1
+$EndComp
+Connection ~ 6100 2600
+Wire Wire Line
+	5600 2500 5700 2500
+Wire Wire Line
+	5700 2500 5700 1900
+Connection ~ 6100 1900
+Wire Wire Line
+	5600 2700 6500 2700
+Wire Wire Line
+	6500 2700 6500 2800
+Wire Wire Line
+	6500 3300 6500 3400
+Wire Wire Line
+	6500 3400 6100 3400
+Wire Wire Line
+	6100 3400 6100 2800
+Wire Wire Line
+	6100 2800 5600 2800
 $EndSCHEMATC

Commit message: Split into separate boards
Parts:
- added C3, C4, C? (x4): 0.1uF, CAPC1608-N, symbol C
- added C5: 0.056uF, CAPC1608-N, symbol C
- added C? (x6): C, ~, symbol C
- added C?: 10uF, ~, symbol C
- added J?: USB_MINI, ~, symbol USB_MINI
- added L? (x2): L, ~, symbol L
- added R? (x8): R, ~, symbol R
- added U? (x2): AOZ1031, ~, symbol AOZ1031
Connections:
- net labels added: +3.3V, +5V, +BATT, CS, D+, D-, GND, INT, MISO, MOSI, OSC1, OSC2, PGC, PGD, SCK, VBus, VCap, XIN, XOUT, ~MCLR
- wire segments 14 -> 120
- no-connect marks 0 -> 1
Other:
- moved on the sheet: C1, C2, L1, U2
