File: Hardware/Wheel Pod Board/Power.sch (KiCad schematic (older format))
At the start: 16 parts

Commit message: More parts on PCB
Parts:
- gave numbers to parts that had none: 16
Changed lines of the file:
@@
 $EndDescr
 $Comp
-L AOZ1280CI U?
+L AOZ1280CI U6
 U 1 1 54F863C5
 P 4700 5200
-F 0 "U?" H 4500 4850 60  0000 C CNN
+F 0 "U6" H 4500 4850 60  0000 C CNN
 F 1 "AOZ1280CI" H 4500 5350 60  0000 C CNN
 F 2 "SMD_Packages:SOT-23-6" H 4700 5200 60  0001 C CNN
@@
 	4850 5300 6050 5300
 $Comp
-L GND #PWR016
+L GND #PWR026
 U 1 1 54F863CD
 P 5650 5900
-F 0 "#PWR016" H 5650 5650 60  0001 C CNN
+F 0 "#PWR026" H 5650 5650 60  0001 C CNN
 F 1 "GND" H 5650 5750 60  0000 C CNN
 F 2 "" H 5650 5900 60  0000 C CNN
@@
 	3100 5300 3200 5300
 $Comp
-L DIODESCH D?
+L DIODESCH D2
 U 1 1 54F863E2
 P 3850 4850
-F 0 "D?" V 3950 5050 60  0000 R CNN
+F 0 "D2" V 3950 5050 60  0000 R CNN
 F 1 "DIODESCH" H 3750 5200 50  0001 C CNN
 F 2 "MAVRIC_footprints:Diode_MicroSMP" H 3850 4850 60  0001 C CNN
@@
 $EndComp
 $Comp
-L GND #PWR017
+L GND #PWR027
 U 1 1 54F863E9
 P 2750 5850
-F 0 "#PWR017" H 2750 5600 60  0001 C CNN
+F 0 "#PWR027" H 2750 5600 60  0001 C CNN
 F 1 "GND" H 2750 5700 60  0000 C CNN
 F 2 "" H 2750 5850 60  0000 C CNN
@@
 	3850 5150 3850 5050
 $Comp
-L GND #PWR018
+L GND #PWR028
 U 1 1 54F863F6
 P 3850 5150
-F 0 "#PWR018" H 3850 4900 60  0001 C CNN
+F 0 "#PWR028" H 3850 4900 60  0001 C CNN
 F 1 "GND" H 3850 5000 60  0000 C CNN
 F 2 "" H 3850 5150 60  0000 C CNN
@@
 Connection ~ 5650 5300
 $Comp
-L Capacitor C?
+L Capacitor C15
 U 1 1 54F8640F
 P 2750 5200
-F 0 "C?" V 2600 5300 60  0000 L CNN
+F 0 "C15" V 2600 5300 60  0000 L CNN
 F 1 "10uF" V 2700 5300 60  0000 L CNN
 F 2 "Capacitors_SMD:C_1206_HandSoldering" H 2650 5200 60  0001 C CNN
@@
 $EndComp
 $Comp
-L Capacitor C?
+L Capacitor C19
 U 1 1 54F8641C
 P 5650 5600
-F 0 "C?" V 5500 5700 60  0000 L CNN
+F 0 "C19" V 5500 5700 60  0000 L CNN
 F 1 "4.7uF" V 5600 5700 60  0000 L CNN
 F 2 "Capacitors_SMD:C_1206_HandSoldering" H 5550 5600 60  0001 C CNN
@@
 	5650 5850 5650 5900
 $Comp
-L Capacitor C?
+L Capacitor C17
 U 1 1 54F8642A
 P 4450 4900
-F 0 "C?" V 4300 5000 60  0000 L CNN
+F 0 "C17" V 4300 5000 60  0000 L CNN
 F 1 "10nF" V 4400 5000 60  0000 L CNN
 F 2 "Capacitors_SMD:C_1206_HandSoldering" H 4350 4900 60  0001 C CNN
@@
 Connection ~ 3100 4550
 $Comp
-L Inductor L?
+L Inductor L2
 U 1 1 54F86439
 P 3500 4550
-F 0 "L?" V 3350 4650 60  0000 L CNN
+F 0 "L2" V 3350 4650 60  0000 L CNN
 F 1 "2.2uH" V 3450 4650 60  0000 L CNN
 F 2 "MAVRIC_footprints:Yuden_SMD_Power_Inductor_6060" H 3400 4550 60  0001 C CNN
@@
 $EndComp
 $Comp
-L Resistor R?
+L Resistor R8
 U 1 1 54F86446
 P 3450 5300
-F 0 "R?" V 3300 5400 60  0000 L CNN
+F 0 "R8" V 3300 5400 60  0000 L CNN
 F 1 "49.9k" V 3400 5400 60  0000 L CNN
 F 2 "Resistors_SMD:R_1206_HandSoldering" H 3350 5300 60  0001 C CNN
@@
 $EndComp
 $Comp
-L Resistor R?
+L Resistor R9
 U 1 1 54F86453
 P 3450 5750
-F 0 "R?" V 3300 5850 60  0000 L CNN
+F 0 "R9" V 3300 5850 60  0000 L CNN
 F 1 "9.53k" V 3400 5850 60  0000 L CNN
 F 2 "Resistors_SMD:R_1206_HandSoldering" H 3350 5750 60  0001 C CNN
@@
 $EndComp
 $Comp
-L +12V #PWR019
+L +12V #PWR029
 U 1 1 54F8645A
 P 6050 1800
-F 0 "#PWR019" H 6050 1650 60  0001 C CNN
+F 0 "#PWR029" H 6050 1650 60  0001 C CNN
 F 1 "+12V" H 6050 1940 60  0000 C CNN
 F 2 "" H 6050 1800 60  0000 C CNN
@@
 $EndComp
 $Comp
-L AOZ1280CI U?
+L AOZ1280CI U5
 U 1 1 54F86460
 P 4700 2550
-F 0 "U?" H 4500 2200 60  0000 C CNN
+F 0 "U5" H 4500 2200 60  0000 C CNN
 F 1 "AOZ1280CI" H 4500 2700 60  0000 C CNN
 F 2 "SMD_Packages:SOT-23-6" H 4700 2550 60  0001 C CNN
@@
 	4850 2650 6050 2650
 $Comp
-L GND #PWR020
+L GND #PWR030
 U 1 1 54F86468
 P 5650 3250
-F 0 "#PWR020" H 5650 3000 60  0001 C CNN
+F 0 "#PWR030" H 5650 3000 60  0001 C CNN
 F 1 "GND" H 5650 3100 60  0000 C CNN
 F 2 "" H 5650 3250 60  0000 C CNN
@@
 	3100 2650 3200 2650
 $Comp
-L DIODESCH D?
+L DIODESCH D1
 U 1 1 54F8647D
 P 3850 2200
-F 0 "D?" V 3950 2400 60  0000 R CNN
+F 0 "D1" V 3950 2400 60  0000 R CNN
 F 1 "DIODESCH" H 3750 2550 50  0001 C CNN
 F 2 "MAVRIC_footprints:Diode_MicroSMP" H 3850 2200 60  0001 C CNN
@@
 $EndComp
 $Comp
-L GND #PWR021
+L GND #PWR031
 U 1 1 54F86484
 P 2750 3200
-F 0 "#PWR021" H 2750 2950 60  0001 C CNN
+F 0 "#PWR031" H 2750 2950 60  0001 C CNN
 F 1 "GND" H 2750 3050 60  0000 C CNN
 F 2 "" H 2750 3200 60  0000 C CNN
@@
 	3850 2500 3850 2400
 $Comp
-L GND #PWR022
+L GND #PWR032
 U 1 1 54F86491
 P 3850 2500
-F 0 "#PWR022" H 3850 2250 60  0001 C CNN
+F 0 "#PWR032" H 3850 2250 60  0001 C CNN
 F 1 "GND" H 3850 2350 60  0000 C CNN
 F 2 "" H 3850 2500 60  0000 C CNN
@@
 Connection ~ 5650 2650
 $Comp
-L Capacitor C?
+L Capacitor C14
 U 1 1 54F864AA
 P 2750 2550
-F 0 "C?" V 2600 2650 60  0000 L CNN
+F 0 "C14" V 2600 2650 60  0000 L CNN
 F 1 "10uF" V 2700 2650 60  0000 L CNN
 F 2 "Capacitors_SMD:C_1206_HandSoldering" H 2650 2550 60  0001 C CNN
@@
 $EndComp
 $Comp
-L Capacitor C?
+L Capacitor C18
 U 1 1 54F864B7
 P 5650 2950
-F 0 "C?" V 5500 3050 60  0000 L CNN
+F 0 "C18" V 5500 3050 60  0000 L CNN
 F 1 "4.7uF" V 5600 3050 60  0000 L CNN
 F 2 "Capacitors_SMD:C_1206_HandSoldering" H 5550 2950 60  0001 C CNN
@@
 	5650 3200 5650 3250
 $Comp
-L Capacitor C?
+L Capacitor C16
 U 1 1 54F864C5
 P 4450 2250
-F 0 "C?" V 4300 2350 60  0000 L CNN
+F 0 "C16" V 4300 2350 60  0000 L CNN
 F 1 "10nF" V 4400 2350 60  0000 L CNN
 F 2 "Capacitors_SMD:C_1206_HandSoldering" H 4350 2250 60  0001 C CNN
@@
 Connection ~ 3100 1900
 $Comp
-L Inductor L?
+L Inductor L1
 U 1 1 54F864D4
 P 3500 1900
-F 0 "L?" V 3350 2000 60  0000 L CNN
+F 0 "L1" V 3350 2000 60  0000 L CNN
 F 1 "2.2uH" V 3450 2000 60  0000 L CNN
 F 2 "MAVRIC_footprints:Yuden_SMD_Power_Inductor_6060" H 3400 1900 60  0001 C CNN
@@
 $EndComp
 $Comp
-L Resistor R?
+L Resistor R6
 U 1 1 54F864E1
 P 3450 2650
-F 0 "R?" V 3300 2750 60  0000 L CNN
+F 0 "R6" V 3300 2750 60  0000 L CNN
 F 1 "49.9k" V 3400 2750 60  0000 L CNN
 F 2 "Resistors_SMD:R_1206_HandSoldering" H 3350 2650 60  0001 C CNN
@@
 $EndComp
 $Comp
-L Resistor R?
+L Resistor R7
 U 1 1 54F864EE
 P 3450 3100
-F 0 "R?" V 3300 3200 60  0000 L CNN
+F 0 "R7" V 3300 3200 60  0000 L CNN
 F 1 "15.8k" V 3400 3200 60  0000 L CNN
 F 2 "Resistors_SMD:R_1206_HandSoldering" H 3350 3100 60  0001 C CNN
